Commit message: added zed

File: kratos_description/urdf/kratos.xacro (robot description, xacro)
@@ -1,9 +1,8 @@
 <?xml version="1.0"?>
-<xacro:include filename="$(find kratos_description)/urdf/kratos_body.xacro"/>
-<xacro:include filename="$(find kratos_description)/urdf/kratos_wheel.xacro"/>
-<robot name="kratos">
-  <!-- BODY -->
+<robot name="kratos" xmlns:xacro="http://www.ros.org/wiki/xacro">
+  <xacro:include filename="$(find kratos_description)/urdf/kratos_body.xacro"/>
+  <xacro:include filename="$(find kratos_description)/urdf/kratos_wheel.xacro"/>
+  <xacro:include filename="$(find zed_wrapper)/urdf/zed_macro.urdf.xacro" />
   <xacro:kratos_body/>
-  <!-- WHEELS -->
   <xacro:kratos_wheel
       name="left_wheel"
@@ -16,3 +15,47 @@
       xyz="0.3 -0.25 0.0"
       rpy="0 0 0"/>
+  <xacro:zed_camera name="zed" model="zed2i">
+    <origin xyz="0 0 0" rpy="0 0 0"/>
+  </xacro:zed_camera>
+<joint name="zed_mount_joint" type="fixed">
+      <parent link="base_link"/>
+      <child link="zed_camera_link"/>
+      <origin xyz="0 0.25 0" rpy="0 0 1.57"/>
+</joint>
+  <gazebo reference="zed_left_camera_frame">
+    <sensor name="zed_camera" type="depth">
+      <visualize>true</visualize>
+      <update_rate>30.0</update_rate>
+      <camera name="zed">
+        <horizontal_fov>1.91986</horizontal_fov>
+        <image>
+          <width>1280</width>
+          <height>720</height>
+          <format>R8G8B8</format>
+        </image>
+        <clip>
+          <near>0.3</near>
+          <far>20.0</far>
+        </clip>
+        <noise>
+          <type>gaussian</type>
+          <mean>0.0</mean>
+          <stddev>0.007</stddev>
+        </noise>
+      </camera>
+      <plugin name="camera_controller" filename="libgazebo_ros_camera.so">
+        <ros>
+          <namespace>zed</namespace>
+          <remapping>zed_camera/image_raw:=zed_node/rgb/image_rect_color</remapping>
+          <remapping>zed_camera/camera_info:=zed_node/rgb/camera_info</remapping>
+          <remapping>zed_camera/depth/image_raw:=zed_node/depth/depth_registered</remapping>
+          <remapping>zed_camera/points:=zed_node/point_cloud/cloud_registered</remapping>
+          <remapping>zed_camera/depth/camera_info:=zed_node/depth/camera_info</remapping>
+        </ros>
+        <frame_name>zed_left_camera_optical_frame</frame_name>
+        <min_depth>0.3</min_depth>
+        <max_depth>20.0</max_depth>
+      </plugin>
+    </sensor>
+  </gazebo>
 </robot>

Commit message: Several Bruh Moments

File: kratos_description/urdf/kratos.xacro (robot description, xacro)
@@ -1,61 +1,50 @@
 <?xml version="1.0"?>
 <robot name="kratos" xmlns:xacro="http://www.ros.org/wiki/xacro">
+  <!-- Define PI constant with higher precision -->
+  <xacro:property name="PI" value="3.14159265359"/>
   <xacro:include filename="$(find kratos_description)/urdf/kratos_body.xacro"/>
-  <xacro:include filename="$(find kratos_description)/urdf/kratos_wheel.xacro"/>
+  <xacro:include filename="$(find kratos_description)/urdf/kratos_left_wheel.xacro"/>
+  <xacro:include filename="$(find kratos_description)/urdf/kratos_right_wheel.xacro"/>
   <xacro:include filename="$(find zed_wrapper)/urdf/zed_macro.urdf.xacro" />
   <xacro:kratos_body/>
-  <xacro:kratos_wheel
-      name="left_wheel"
+  <!-- Left side wheels (3 wheels) -->
+  <xacro:kratos_left_wheel
+      name="left_wheel_front"
       parent="base_link"
-      xyz="0.3 0.25 0.0"
+      xyz="0.4 0.5 0.0"
       rpy="0 0 0"/>
-  <xacro:kratos_wheel
-      name="right_wheel"
+  <xacro:kratos_left_wheel
+      name="left_wheel_middle"
       parent="base_link"
-      xyz="0.3 -0.25 0.0"
+      xyz="0.0 0.5 0.0"
+      rpy="0 0 0"/>
+  <xacro:kratos_left_wheel
+      name="left_wheel_rear"
+      parent="base_link"
+      xyz="-0.4 0.5 0.0"
+      rpy="0 0 0"/>
+  <!-- Right side wheels (3 wheels) -->
+  <xacro:kratos_right_wheel
+      name="right_wheel_front"
+      parent="base_link"
+      xyz="0.4 -0.5 0.0"
+      rpy="0 0 0"/>
+  <xacro:kratos_right_wheel
+      name="right_wheel_middle"
+      parent="base_link"
+      xyz="0.0 -0.5 0.0"
+      rpy="0 0 0"/>
+  <xacro:kratos_right_wheel
+      name="right_wheel_rear"
+      parent="base_link"
+      xyz="-0.4 -0.5 0.0"
       rpy="0 0 0"/>
   <xacro:zed_camera name="zed" model="zed2i">
     <origin xyz="0 0 0" rpy="0 0 0"/>
   </xacro:zed_camera>
-<joint name="zed_mount_joint" type="fixed">
-      <parent link="base_link"/>
-      <child link="zed_camera_link"/>
-      <origin xyz="0 0.25 0" rpy="0 0 1.57"/>
-</joint>
-  <gazebo reference="zed_left_camera_frame">
-    <sensor name="zed_camera" type="depth">
-      <visualize>true</visualize>
-      <update_rate>30.0</update_rate>
-      <camera name="zed">
-        <horizontal_fov>1.91986</horizontal_fov>
-        <image>
-          <width>1280</width>
-          <height>720</height>
-          <format>R8G8B8</format>
-        </image>
-        <clip>
-          <near>0.3</near>
-          <far>20.0</far>
-        </clip>
-        <noise>
-          <type>gaussian</type>
-          <mean>0.0</mean>
-          <stddev>0.007</stddev>
-        </noise>
-      </camera>
-      <plugin name="camera_controller" filename="libgazebo_ros_camera.so">
-        <ros>
-          <namespace>zed</namespace>
-          <remapping>zed_camera/image_raw:=zed_node/rgb/image_rect_color</remapping>
-          <remapping>zed_camera/camera_info:=zed_node/rgb/camera_info</remapping>
-          <remapping>zed_camera/depth/image_raw:=zed_node/depth/depth_registered</remapping>
-          <remapping>zed_camera/points:=zed_node/point_cloud/cloud_registered</remapping>
-          <remapping>zed_camera/depth/camera_info:=zed_node/depth/camera_info</remapping>
-        </ros>
-        <frame_name>zed_left_camera_optical_frame</frame_name>
-        <min_depth>0.3</min_depth>
-        <max_depth>20.0</max_depth>
-      </plugin>
-    </sensor>
-  </gazebo>
+  <joint name="zed_mount_joint" type="fixed">
+    <parent link="base_link"/>
+    <child link="zed_camera_link"/>
+    <origin xyz="0 0.25 0" rpy="0 0 ${-PI/2}"/>
+  </joint>
 </robot>

File: kratos_description/urdf/kratos_body.xacro (robot description, xacro)
@@ -1,9 +1,11 @@
 <?xml version="1.0"?>
 <robot xmlns:xacro="http://www.ros.org/wiki/xacro">
+  <!-- Define PI constant -->
+  <xacro:property name="PI" value="3.14159265359"/>
   <xacro:macro name="kratos_body">
     <link name="base_link">
       <!-- Visual -->
       <visual>
-        <origin xyz="0 0 0" rpy="0 0 0"/>
+        <origin xyz="0 0 0" rpy="0 0 ${-PI/2}"/>
         <geometry>
           <mesh filename="package://kratos_description/meshes/body.stl"

File: kratos_gazebo/urdf/kratos.gazebo.xacro (robot description, xacro)
@@ -14,6 +14,6 @@
     <kd>1.0</kd>  <!-- Contact damping -->
   </gazebo>
-  <!-- Gazebo properties for left wheel -->
-  <gazebo reference="left_wheel">
+  <!-- Gazebo properties for left wheels -->
+  <gazebo reference="left_wheel_front">
     <material>Gazebo/Black</material>
     <mu1>1.0</mu1>  <!-- Higher friction for wheels -->
@@ -22,6 +22,34 @@
     <kd>1.0</kd>
   </gazebo>
-  <!-- Gazebo properties for right wheel -->
-  <gazebo reference="right_wheel">
+  <gazebo reference="left_wheel_middle">
+    <material>Gazebo/Black</material>
+    <mu1>1.0</mu1>
+    <mu2>1.0</mu2>
+    <kp>1000000.0</kp>
+    <kd>1.0</kd>
+  </gazebo>
+  <gazebo reference="left_wheel_rear">
+    <material>Gazebo/Black</material>
+    <mu1>1.0</mu1>
+    <mu2>1.0</mu2>
+    <kp>1000000.0</kp>
+    <kd>1.0</kd>
+  </gazebo>
+  <!-- Gazebo properties for right wheels -->
+  <gazebo reference="right_wheel_front">
+    <material>Gazebo/Black</material>
+    <mu1>1.0</mu1>
+    <mu2>1.0</mu2>
+    <kp>1000000.0</kp>
+    <kd>1.0</kd>
+  </gazebo>
+  <gazebo reference="right_wheel_middle">
+    <material>Gazebo/Black</material>
+    <mu1>1.0</mu1>
+    <mu2>1.0</mu2>
+    <kp>1000000.0</kp>
+    <kd>1.0</kd>
+  </gazebo>
+  <gazebo reference="right_wheel_rear">
     <material>Gazebo/Black</material>
     <mu1>1.0</mu1>
@@ -34,13 +62,20 @@
   <!-- ========================================= -->
   <!-- Differential drive plugin for robot control -->
+  <!-- FIXED: Only use middle wheels (one left, one right) -->
   <gazebo>
     <plugin name="differential_drive_controller" filename="libgazebo_ros_diff_drive.so">
+      <!-- ROS 2 Configuration -->
+      <ros>
+        <namespace>/</namespace>
+        <remapping>cmd_vel:=cmd_vel</remapping>
+        <remapping>odom:=odom</remapping>
+      </ros>
       <!-- Update rate in Hz -->
       <update_rate>50</update_rate>
-      <!-- Wheel joints -->
-      <left_joint>left_wheel_joint</left_joint>
-      <right_joint>right_wheel_joint</right_joint>
+      <!-- Only middle wheels are driven (one left, one right) -->
+      <left_joint>left_wheel_middle_joint</left_joint>
+      <right_joint>right_wheel_middle_joint</right_joint>
       <!-- Kinematics -->
-      <wheel_separation>0.5</wheel_separation>  <!-- Distance between wheels -->
+      <wheel_separation>0.5</wheel_separation>  <!-- Distance between left and right wheels (Y-axis) -->
       <wheel_diameter>0.2</wheel_diameter>  <!-- Wheel diameter -->
       <!-- Limits -->
@@ -53,8 +88,4 @@
       <odometry_frame>odom</odometry_frame>
       <robot_base_frame>base_link</robot_base_frame>
-      <!-- Topic to receive velocity commands -->
-      <command_topic>cmd_vel</command_topic>
-      <!-- Topic to publish odometry -->
-      <odometry_topic>odom</odometry_topic>
     </plugin>
   </gazebo>
@@ -62,8 +93,88 @@
   <gazebo>
     <plugin name="gazebo_ros_joint_state_publisher" filename="libgazebo_ros_joint_state_publisher.so">
+      <ros>
+        <namespace>/</namespace>
+      </ros>
       <update_rate>50</update_rate>
-      <joint_name>left_wheel_joint</joint_name>
-      <joint_name>right_wheel_joint</joint_name>
+      <joint_name>left_wheel_front_joint</joint_name>
+      <joint_name>left_wheel_middle_joint</joint_name>
+      <joint_name>left_wheel_rear_joint</joint_name>
+      <joint_name>right_wheel_front_joint</joint_name>
+      <joint_name>right_wheel_middle_joint</joint_name>
+      <joint_name>right_wheel_rear_joint</joint_name>
     </plugin>
   </gazebo>
+  <!-- ========================================= -->
+  <!-- ZED CAMERA GAZEBO SENSOR CONFIGURATION -->
+  <!-- ========================================= -->
+  <!-- ZED camera sensor configuration for Gazebo -->
+  <gazebo reference="zed_left_camera_frame">
+    <sensor name="zed_camera" type="depth">
+      <visualize>false</visualize>
+      <update_rate>10.0</update_rate>
+      <camera name="zed">
+        <horizontal_fov>1.91986</horizontal_fov>
+        <image>
+          <width>640</width>
+          <height>480</height>
+          <format>R8G8B8</format>
+        </image>
+        <clip>
+          <near>0.3</near>
+          <far>20.0</far>
+        </clip>
+        <noise>
+          <type>gaussian</type>
+          <mean>0.0</mean>
+          <stddev>0.007</stddev>
+        </noise>
+      </camera>
+      <plugin name="camera_controller" filename="libgazebo_ros_camera.so">
+        <ros>
+          <namespace>zed</namespace>
+          <remapping>zed_camera/image_raw:=zed_node/rgb/image_rect_color</remapping>
+          <remapping>zed_camera/camera_info:=zed_node/rgb/camera_info</remapping>
+          <remapping>zed_camera/depth/image_raw:=zed_node/depth/depth_registered</remapping>
+          <remapping>zed_camera/points:=zed_node/point_cloud/cloud_registered</remapping>
+          <remapping>zed_camera/depth/camera_info:=zed_node/depth/camera_info</remapping>
+        </ros>
+        <frame_name>zed_left_camera_optical_frame</frame_name>
+        <min_depth>0.3</min_depth>
+        <max_depth>20.0</max_depth>
+        <!-- Queue size and performance settings -->
+        <ros>
+          <qos>
+            <topic name="zed_node/rgb/image_rect_color">
+              <publisher>
+                <reliability>best_effort</reliability>
+                <durability>volatile</durability>
+                <deadline>
+                  <sec>0</sec>
+                  <nsec>100000000</nsec>
+                </deadline>
+                <lifespan>
+                  <sec>1</sec>
+                  <nsec>0</nsec>
+                </lifespan>
+              </publisher>
+            </topic>
+            <topic name="zed_node/depth/depth_registered">
+              <publisher>
+                <reliability>best_effort</reliability>
+                <durability>volatile</durability>
+                <deadline>
+                  <sec>0</sec>
+                  <nsec>100000000</nsec>
+                </deadline>
+                <lifespan>
+                  <sec>1</sec>
+                  <nsec>0</nsec>
+                </lifespan>
+              </publisher>
+            </topic>
+          </qos>
+        </ros>
+      </plugin>
+    </sensor>
+  </gazebo>
 </robot>

Commit message: Fixed Zed Added Cones

File: kratos_description/urdf/kratos.xacro (robot description, xacro)
@@ -46,5 +46,5 @@
     <parent link="base_link"/>
     <child link="zed_camera_link"/>
-    <origin xyz="0 0.25 0" rpy="0 0 ${-PI/2}"/>
+    <origin xyz="0.25 0 0" rpy="0 0 0"/>
   </joint>
 </robot>
